File: pcb/christmas-tree-pcb.kicad_pcb (KiCad board)
At the start: 2 copper layers, 56.1 x 89.5 mm, 17 parts, among them SW1 SS12D00G, U1 ATtiny202-SS

Commit message: PCB layout; Comply with DRC
Other:
- board text added: "Happy Holidays!"
- board text removed: "Joyeux Noël et bonne année !"
